Commit message: simulation

File: src/pkg/rover_description_pkg/urdf/rover_macro.xacro (robot description, xacro)
@@ -90,5 +90,5 @@
             <parent link="payload_link"/>
             <child link="${laser_frame}"/>
-            <origin xyz="0.075 0 -0.01" rpy="0.0 0.0 3.1415"/>
+            <origin xyz="0.075 0 -0.01" rpy="0.0 0.0 0.0"/>
         </joint>
         <link name="${laser_frame}">
